File: hardware/devboard/LPC11Uxx_dev_board_frame.kicad_pcb (KiCad board)
At the start: 2 copper layers, 58.9 x 53 mm, 41 parts, among them J1 Conn_ARM_JTAG_SWD_10, J2 USB_B_Micro, J3 Conn_01x04_Male, J4 Conn_01x16_Male, J5 Conn_01x16_Male, Q1 DMP2035U, Q2 DMP2035U, SW1 SW_Push, U1 LPC11U37FBD48-401_, U2 MCP1825S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

Commit message: Devboard PCB: Fix frame tooling hole-to-hole distance to multiple of 20mm
Parts:
- moved REF** 71.3 mm to (38.6, 28.6), turned to 180 degrees
- moved REF** 69.3 mm to (38.6, 68.6), turned to 180 degrees
- moved REF** 69.1 mm to (98.6, 28.6), turned to 180 degrees
- moved REF** 67.1 mm to (98.6, 68.6), turned to 180 degrees
Other:
- board size 58.9 x 53 mm -> 66 x 53 mm
Changed lines of the file:
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@@
-(kicad_pcb (version 20171130) (host pcbnew "(5.0.1-3-g963ef8bb5)")
+(kicad_pcb (version 20171130) (host pcbnew 5.0.2-bee76a0~70~ubuntu18.04.1)
   (general
     (thickness 1.6)
@@
     (visible_elements FFFFFF7F)
     (pcbplotparams
-      (layerselection 0x010fc_ffffffff)
+      (layerselection 0x010f0_ffffffff)
       (usegerberextensions false)
       (usegerberattributes false)
@@
   )
   (module Jitter_Footprints:Tooling_hole_4mm_4.04mm_paste locked (layer F.Cu)
-    (at 96.4 70.3)
-    (fp_text reference REF** (at -4.8 -1.5) (layer F.SilkS) hide
-      (effects (font (size 1 1) (thickness 0.15)))
-    )
-    (fp_text value "Tooling hole 4mm_4.04mm_paste" (at 0 -3.2) (layer F.Fab) hide
-      (effects (font (size 1 1) (thickness 0.15)))
-    )
-    (pad "" np_thru_hole circle (at 0 0) (size 4 4) (drill 4) (layers *.Cu *.Mask F.Paste)
+    (at 38.6 28.6 180)
+    (fp_text reference REF** (at -4.8 -1.5 180) (layer F.SilkS) hide
+      (effects (font (size 1 1) (thickness 0.15)))
+    )
+    (fp_text value "Tooling hole 4mm_4.04mm_paste" (at 0 -3.2 180) (layer F.Fab) hide
+      (effects (font (size 1 1) (thickness 0.15)))
+    )
+    (pad "" np_thru_hole circle (at 0 0 180) (size 4 4) (drill 4) (layers *.Cu *.Mask F.Paste)
       (solder_paste_margin 0.04))
   )
   (module Jitter_Footprints:Tooling_hole_4mm_4.04mm_paste locked (layer F.Cu)
-    (at 96.4 30.3)
-    (fp_text reference REF** (at -4.8 -1.5) (layer F.SilkS) hide
-      (effects (font (size 1 1) (thickness 0.15)))
-    )
-    (fp_text value "Tooling hole 4mm_4.04mm_paste" (at 0 -3.2) (layer F.Fab) hide
-      (effects (font (size 1 1) (thickness 0.15)))
-    )
-    (pad "" np_thru_hole circle (at 0 0) (size 4 4) (drill 4) (layers *.Cu *.Mask F.Paste)
+    (at 38.6 68.6 180)
+    (fp_text reference REF** (at -4.8 -1.5 180) (layer F.SilkS) hide
+      (effects (font (size 1 1) (thickness 0.15)))
+    )
+    (fp_text value "Tooling hole 4mm_4.04mm_paste" (at 0 -3.2 180) (layer F.Fab) hide
+      (effects (font (size 1 1) (thickness 0.15)))
+    )
+    (pad "" np_thru_hole circle (at 0 0 180) (size 4 4) (drill 4) (layers *.Cu *.Mask F.Paste)
       (solder_paste_margin 0.04))
   )
   (module Jitter_Footprints:Tooling_hole_4mm_4.04mm_paste locked (layer F.Cu)
-    (at 43.5 30.3)
-    (fp_text reference REF** (at -4.8 -1.5) (layer F.SilkS) hide
-      (effects (font (size 1 1) (thickness 0.15)))
-    )
-    (fp_text value "Tooling hole 4mm_4.04mm_paste" (at 0 -3.2) (layer F.Fab) hide
-      (effects (font (size 1 1) (thickness 0.15)))
-    )
-    (pad "" np_thru_hole circle (at 0 0) (size 4 4) (drill 4) (layers *.Cu *.Mask F.Paste)
+    (at 98.6 68.6 180)
+    (fp_text reference REF** (at -4.8 -1.5 180) (layer F.SilkS) hide
+      (effects (font (size 1 1) (thickness 0.15)))
+    )
+    (fp_text value "Tooling hole 4mm_4.04mm_paste" (at 0 -3.2 180) (layer F.Fab) hide
+      (effects (font (size 1 1) (thickness 0.15)))
+    )
+    (pad "" np_thru_hole circle (at 0 0 180) (size 4 4) (drill 4) (layers *.Cu *.Mask F.Paste)
       (solder_paste_margin 0.04))
   )
   (module Jitter_Footprints:Tooling_hole_4mm_4.04mm_paste locked (layer F.Cu)
-    (at 43.5 70.3)
-    (fp_text reference REF** (at -4.8 -1.5) (layer F.SilkS) hide
-      (effects (font (size 1 1) (thickness 0.15)))
-    )
-    (fp_text value "Tooling hole 4mm_4.04mm_paste" (at 0 -3.2) (layer F.Fab) hide
-      (effects (font (size 1 1) (thickness 0.15)))
-    )
-    (pad "" np_thru_hole circle (at 0 0) (size 4 4) (drill 4) (layers *.Cu *.Mask F.Paste)
+    (at 98.6 28.6 180)
+    (fp_text reference REF** (at -4.8 -1.5 180) (layer F.SilkS) hide
+      (effects (font (size 1 1) (thickness 0.15)))
+    )
+    (fp_text value "Tooling hole 4mm_4.04mm_paste" (at 0 -3.2 180) (layer F.Fab) hide
+      (effects (font (size 1 1) (thickness 0.15)))
+    )
+    (pad "" np_thru_hole circle (at 0 0 180) (size 4 4) (drill 4) (layers *.Cu *.Mask F.Paste)
       (solder_paste_margin 0.04))
   )
@@
   (gr_line (start 46.3 37.1) (end 46.3 63.95) (layer Edge.Cuts) (width 0.15))
   (gr_line (start 48.5 37.1) (end 48.5 63.95) (layer Edge.Cuts) (width 0.15))
-  (gr_line (start 46.3 67.55) (end 46.3 73.3) (layer Edge.Cuts) (width 0.15))
+  (gr_line (start 46.3 67.55) (end 46.3 75.3) (layer Edge.Cuts) (width 0.15))
   (gr_line (start 48.5 67.55) (end 48.5 73.3) (layer Edge.Cuts) (width 0.15))
-  (gr_line (start 93.2 67.55) (end 93.2 73.3) (layer Edge.Cuts) (width 0.15))
+  (gr_line (start 93.2 67.55) (end 93.2 75.3) (layer Edge.Cuts) (width 0.15))
   (gr_line (start 91 63.95) (end 91 37.05) (layer Edge.Cuts) (width 0.15))
   (gr_line (start 93.2 37.05) (end 93.2 63.95) (layer Edge.Cuts) (width 0.15))
@@
   (gr_line (start 46.3 37.1) (end 48.5 37.1) (layer Edge.Cuts) (width 0.15))
   (gr_line (start 46.3 33.5) (end 48.5 33.5) (layer Edge.Cuts) (width 0.15))
-  (gr_line (start 93.2 27.2) (end 93.2 33.45) (layer Edge.Cuts) (width 0.15))
-  (gr_line (start 99.2 27.2) (end 99.2 73.3) (layer Edge.Cuts) (width 0.15))
-  (gr_line (start 93.2 27.2) (end 99.2 27.2) (layer Edge.Cuts) (width 0.15))
-  (gr_line (start 93.2 73.3) (end 99.2 73.3) (layer Edge.Cuts) (width 0.15))
-  (gr_line (start 40.3 27.2) (end 46.3 27.2) (layer Edge.Cuts) (width 0.15))
-  (gr_line (start 40.3 73.3) (end 46.3 73.3) (layer Edge.Cuts) (width 0.15))
-  (gr_line (start 40.3 27.2) (end 40.3 73.3) (layer Edge.Cuts) (width 0.15))
+  (gr_line (start 93.2 22.3) (end 93.2 33.45) (layer Edge.Cuts) (width 0.15))
+  (gr_line (start 101.5 22.3) (end 101.5 75.3) (layer Edge.Cuts) (width 0.15))
+  (gr_line (start 93.2 22.3) (end 101.5 22.3) (layer Edge.Cuts) (width 0.15))
+  (gr_line (start 93.2 75.3) (end 101.5 75.3) (layer Edge.Cuts) (width 0.15))
+  (gr_line (start 35.5 22.3) (end 46.3 22.3) (layer Edge.Cuts) (width 0.15))
+  (gr_line (start 35.5 75.3) (end 46.3 75.3) (layer Edge.Cuts) (width 0.15))
+  (gr_line (start 35.5 22.3) (end 35.5 75.3) (layer Edge.Cuts) (width 0.15))
   (target plus (at 48.504208 75.294393) (size 5) (width 0.15) (layer Edge.Cuts))
-  (gr_line (start 46.3 27.2) (end 46.3 33.5) (layer Edge.Cuts) (width 0.15))
+  (gr_line (start 46.3 22.3) (end 46.3 33.5) (layer Edge.Cuts) (width 0.15))
   (gr_line (start 48.5 24.3) (end 48.5 33.5) (layer Edge.Cuts) (width 0.15))
   (gr_line (start 91 73.3) (end 91 67.55) (layer Edge.Cuts) (width 0.15))
