File: hardware/devboard/LPC11Uxx_dev_board.sch (KiCad schematic (older format))
At the start: 31 parts, among them J1 Conn_ARM_JTAG_SWD_10, J2 USB_B_Micro, J3 Conn_01x04_Male, J4 Conn_01x16_Male, J5 Conn_01x16_Male, Q1 DMP2035U, Q2 DMP2035U, SW1 SW_Push, U1 LPC11U37FBD48-401_, U2 MCP1825S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

Commit message: Pick diode
Parts:
- D3: value D -> NRVTS245ESF
Other:
- note removed: "TODO: Pick diode"
Changed lines of the file:
@@
 P 2050 5800
 F 0 "D3" H 2150 5650 50  0000 C CNN
-F 1 "D" H 2050 5650 50  0000 C CNN
+F 1 "NRVTS245ESF" H 2050 5650 50  0000 C CNN
 F 2 "Diode_SMD:D_SOD-123F" H 2050 5800 50  0001 C CNN
-F 3 "~" H 2050 5800 50  0001 C CNN
+F 3 "http://www.farnell.com/datasheets/1900855.pdf" H 2050 5800 50  0001 C CNN
 	1    2050 5800
 	1    0    0    -1
@@
 Wire Wire Line
 	2000 2950 2100 2950
-Text Notes 1900 6100 0    50   ~ 0
-TODO: Pick diode
 Wire Wire Line
 	1150 3900 1150 4000

Commit message: Update some components for lpc11
Parts:
- J1: symbol Connector:Conn_ARM_JTAG_SWD_10 -> LPC11Uxx_dev_board-rescue:Conn_ARM_JTAG_SWD_10-Connector
- SW1: value SW_Push -> EVQPE1
Changed lines of the file:
@@
 EESchema Schematic File Version 4
 LIBS:LPC11Uxx_dev_board-cache
-EELAYER 26 0
+EELAYER 29 0
 EELAYER END
 $Descr A4 11693 8268
@@
 	3400 3650 3850 3650
 $Comp
-L Connector:Conn_ARM_JTAG_SWD_10 J1
+L LPC11Uxx_dev_board-rescue:Conn_ARM_JTAG_SWD_10-Connector J1
 U 1 1 5B913C24
 P 9300 2600
@@
 P 7350 950
 F 0 "SW1" H 7350 1235 50  0000 C CNN
-F 1 "SW_Push" H 7350 1144 50  0000 C CNN
+F 1 "EVQPE1" H 7350 1144 50  0000 C CNN
 F 2 "Button_Switch_SMD:SW_SPST_EVQPE1" H 7350 1150 50  0001 C CNN
 F 3 "" H 7350 1150 50  0001 C CNN
