File: hardware/Breakout/lpc11_breakout.kicad_pcb (KiCad board)
At the start: 2 copper layers, 48.3 x 48.3 mm, 24 parts, among them J1 Conn_01x04_Male, J2 Conn_02x04_Odd_Even, J3 Conn_02x12_Odd_Even, J4 Conn_02x12_Odd_Even, J5 Conn_02x12_Odd_Even, J6 Conn_02x04_Odd_Even, U1 LPC1115JBD48-303, Y1 MCSJK-7U-12.00-10-10-80-B-10

Commit message: Fix bug on LPC11 breakout board: SWDIO pin
Parts:
- renumbered RST to SW1
Connections:
- J1 pad 2: /SWDIO_35 -> /SWDIO_39
- J5 pad 9: /39 -> /SWDIO_39
- J6 pad 5: /SWDIO_35 -> /35
- U1 pad 35: /SWDIO_35 -> /35
- U1 pad 39: /39 -> /SWDIO_39
Routing:
- net /SWDIO_39: track 0.00 -> 53.2 mm
- net /SWDIO_35: track 36.2 -> 0.00 mm
- net /35: track 0.00 -> 18.5 mm
- net /39: track 15.6 -> 0.00 mm
- net +3V3: track 66.2 -> 61.5 mm
